File: RS-MINI-ULTRA-8M.sch (KiCad schematic (older format))
At the start: 24 parts, among them J1 2.54 mm 1x6, J2 2.54 mm 1x14, J3 2.54 mm 1x14, M1 FIDUCIAL, M2 FIDUCIAL, Q1 2N7002, SW1 SPNO, U1 MCP1700T-3302E/MB, U2 ATMEGA328P-AU, Y1 PBRC8.00MR50X000

Commit message: Version 1.60
Other:
- note added: "FTDI Header"
- note added: "Logos"
- note added: "Pin Breakout"
- moved on the sheet: C6, D2, J1, J2, J3, Q1, R2
